File: modul_16_segment_LED/mod_16_segment_LED.sch (KiCad schematic (older format))
At the start: 28 parts

Commit message: Добавил таблицу для подключения платы 16_segment_LED к SPI.
Other:
- note added: "SPI SafeDuino SafeDuino 2560\n\nDS MOSI 14 MOSI\n\nSHCP SCK 13 SCK\n\nSTCP CS 8 8"
- note added: "Подключение платы к интерфейсу SPI"
Changed lines of the file:
@@
-EESchema Schematic File Version 2  date Fri 19 Jul 2013 13:04:34 MSK
-LIBS:LFbutton
-LIBS:LFcapitors
-LIBS:LFcomponents
-LIBS:LFconnectors
-LIBS:LFdiod
-LIBS:LFpower
-LIBS:LFresistor
-LIBS:LFtransformator
-LIBS:LFtransistor
+EESchema Schematic File Version 2
 LIBS:mod_16_segment_LED-cache
-EELAYER 25  0
+EELAYER 27 0
 EELAYER END
-$Descr A3 16535 11700
+$Descr A3 16535 11693
 encoding utf-8
 Sheet 1 1
 Title ""
-Date "19 jul 2013"
+Date "21 jan 2016"
 Rev ""
 Comp ""
@@
 F 0 "R12" H 6600 7050 71  0000 C CNN
 F 1 "220" H 7150 7050 71  0000 C CNN
+F 2 "" H 6750 7000 60  0001 C CNN
+F 3 "" H 6750 7000 60  0001 C CNN
 	1    6750 7000
 	1    0    0    -1
@@
 F 0 "C4" H 10775 7025 71  0000 C CNN
 F 1 "0.1 мк" H 10775 6925 71  0000 C CNN
+F 2 "" H 10650 6750 60  0001 C CNN
+F 3 "" H 10650 6750 60  0001 C CNN
 	1    10650 6750
 	1    0    0    -1
@@
 F 0 "C5" H 10775 7475 71  0000 C CNN
 F 1 "0.1 мк" H 10775 7375 71  0000 C CNN
+F 2 "" H 10650 7200 60  0001 C CNN
+F 3 "" H 10650 7200 60  0001 C CNN
 	1    10650 7200
 	1    0    0    -1
@@
 F 0 "DD5" H 5450 8750 70  0000 C CNN
 F 1 "74HC595B" H 5600 8600 70  0000 C CNN
+F 2 "" H 5600 8200 60  0001 C CNN
+F 3 "" H 5600 8200 60  0001 C CNN
 	1    5600 8200
 	1    0    0    -1
@@
 F 0 "R11" H 7300 5800 71  0000 C CNN
 F 1 "220" H 7850 5800 71  0000 C CNN
+F 2 "" H 7450 5750 60  0001 C CNN
+F 3 "" H 7450 5750 60  0001 C CNN
 	1    7450 5750
 	1    0    0    -1
@@
 F 0 "R13" H 6650 8050 71  0000 C CNN
 F 1 "220" H 7200 8050 71  0000 C CNN
+F 2 "" H 6800 8000 60  0001 C CNN
+F 3 "" H 6800 8000 60  0001 C CNN
 	1    6800 8000
 	1    0    0    -1
@@
 F 0 "DD4" H 5450 7050 70  0000 C CNN
 F 1 "74HC595B" H 5600 6900 70  0000 C CNN
+F 2 "" H 5600 6500 60  0001 C CNN
+F 3 "" H 5600 6500 60  0001 C CNN
 	1    5600 6500
 	1    0    0    -1
@@
 F 0 "R10" H 6600 5200 71  0000 C CNN
 F 1 "220" H 7150 5200 71  0000 C CNN
+F 2 "" H 6750 5150 60  0001 C CNN
+F 3 "" H 6750 5150 60  0001 C CNN
 	1    6750 5150
 	1    0    0    -1
@@
 F 0 "R9" H 7300 5100 71  0000 C CNN
 F 1 "220" H 7850 5100 71  0000 C CNN
+F 2 "" H 7450 5050 60  0001 C CNN
+F 3 "" H 7450 5050 60  0001 C CNN
 	1    7450 5050
 	1    0    0    -1
@@
 F 0 "R8" H 6600 4800 71  0000 C CNN
 F 1 "220" H 7150 4800 71  0000 C CNN
+F 2 "" H 6750 4750 60  0001 C CNN
+F 3 "" H 6750 4750 60  0001 C CNN
 	1    6750 4750
 	1    0    0    -1
@@
 F 0 "R7" H 7300 4700 71  0000 C CNN
 F 1 "220" H 7850 4700 71  0000 C CNN
+F 2 "" H 7450 4650 60  0001 C CNN
+F 3 "" H 7450 4650 60  0001 C CNN
 	1    7450 4650
 	1    0    0    -1
@@
 F 0 "DPY2" H 9100 5750 60  0000 C CNN
 F 1 "PSA12-11SRWA" H 9350 5650 60  0000 C CNN
+F 2 "" H 9450 5050 60  0001 C CNN
+F 3 "" H 9450 5050 60  0001 C CNN
 	1    9450 5050
 	1    0    0    -1
@@
 F 0 "C3" H 10775 6575 71  0000 C CNN
 F 1 "0.1 мк" H 10775 6475 71  0000 C CNN
+F 2 "" H 10650 6300 60  0001 C CNN
+F 3 "" H 10650 6300 60  0001 C CNN
 	1    10650 6300
 	1    0    0    -1
@@
 F 0 "C2" H 10775 6125 71  0000 C CNN
 F 1 "0.1 мк" H 10775 6025 71  0000 C CNN
+F 2 "" H 10650 5850 60  0001 C CNN
+F 3 "" H 10650 5850 60  0001 C CNN
 	1    10650 5850
 	1    0    0    -1
@@
 F 0 "C1" H 10775 5675 71  0000 C CNN
 F 1 "0.1 мк" H 10775 5575 71  0000 C CNN
+F 2 "" H 10650 5400 60  0001 C CNN
+F 3 "" H 10650 5400 60  0001 C CNN
 	1    10650 5400
 	1    0    0    -1
@@
 F 0 "R14" H 7300 8150 71  0000 C CNN
 F 1 "220" H 7850 8150 71  0000 C CNN
+F 2 "" H 7450 8100 60  0001 C CNN
+F 3 "" H 7450 8100 60  0001 C CNN
 	1    7450 8100
 	1    0    0    -1
@@
 F 0 "DD3" H 5500 5400 70  0000 C CNN
 F 1 "74HC595B" H 5650 5250 70  0000 C CNN
+F 2 "" H 5650 4850 60  0001 C CNN
+F 3 "" H 5650 4850 60  0001 C CNN
 	1    5650 4850
 	1    0    0    -1
@@
 F 1 "PBS-5R" H 10800 3200 50  0000 L BNN
 F 2 "~" H 11200 3250 50  0001 C CNN
+F 3 "" H 10750 3100 60  0001 C CNN
 	1    10750 3100
 	1    0    0    -1
@@
 F 0 "R5" H 7300 2550 71  0000 C CNN
 F 1 "220" H 7900 2550 71  0000 C CNN
+F 2 "" H 7450 2500 60  0001 C CNN
+F 3 "" H 7450 2500 60  0001 C CNN
 	1    7450 2500
 	1    0    0    -1
@@
 F 0 "R1" H 6600 1450 71  0000 C CNN
 F 1 "220" H 7200 1450 71  0000 C CNN
+F 2 "" H 6750 1400 60  0001 C CNN
+F 3 "" H 6750 1400 60  0001 C CNN
 	1    6750 1400
 	1    0    0    -1
@@
 F 0 "R6" H 6600 3750 71  0000 C CNN
 F 1 "220" H 7150 3750 71  0000 C CNN
+F 2 "" H 6750 3700 60  0001 C CNN
+F 3 "" H 6750 3700 60  0001 C CNN
 	1    6750 3700
 	1    0    0    -1
@@
 F 0 "R4" H 7300 1950 71  0000 C CNN
 F 1 "220" H 7900 1950 71  0000 C CNN
+F 2 "" H 7450 1900 60  0001 C CNN
+F 3 "" H 7450 1900 60  0001 C CNN
 	1    7450 1900
 	1    0    0    -1
@@
 F 0 "R3" H 6600 1850 71  0000 C CNN
 F 1 "220" H 7200 1850 71  0000 C CNN
+F 2 "" H 6750 1800 60  0001 C CNN
+F 3 "" H 6750 1800 60  0001 C CNN
 	1    6750 1800
 	1    0    0    -1
@@
 F 0 "R2" H 7300 1550 71  0000 C CNN
 F 1 "220" H 7900 1550 71  0000 C CNN
+F 2 "" H 7450 1500 60  0001 C CNN
+F 3 "" H 7450 1500 60  0001 C CNN
 	1    7450 1500
 	1    0    0    -1
@@
 F 0 "DPY1" H 9100 2500 60  0000 C CNN
 F 1 "PSA12-11SRWA" H 9350 2400 60  0000 C CNN
+F 2 "" H 9450 1800 60  0001 C CNN
+F 3 "" H 9450 1800 60  0001 C CNN
 	1    9450 1800
 	1    0    0    -1
@@
 F 1 "PLS-5/PLS2-5R" H 2650 3200 50  0000 L BNN
 F 2 "~" H 3200 3250 50  0001 C CNN
+F 3 "" H 2750 3100 60  0001 C CNN
 	1    2750 3100
 	-1   0    0    -1
@@
 F 0 "DD2" H 5500 3750 70  0000 C CNN
 F 1 "74HC595B" H 5650 3600 70  0000 C CNN
+F 2 "" H 5650 3200 60  0001 C CNN
+F 3 "" H 5650 3200 60  0001 C CNN
 	1    5650 3200
 	1    0    0    -1
@@
 F 0 "DD1" H 5500 2150 70  0000 C CNN
 F 1 "74HC595B" H 5650 2000 70  0000 C CNN
+F 2 "" H 5650 1600 60  0001 C CNN
+F 3 "" H 5650 1600 60  0001 C CNN
 	1    5650 1600
 	1    0    0    -1
 $EndComp
+Text Notes 1250 9600 0    60   ~ 0
+           SPI        SafeDuino    SafeDuino 2560\n\nDS        MOSI         14            MOSI\n\nSHCP      SCK         13             SCK\n\nSTCP       CS           8               8
+Wire Notes Line
+	1250 9800 3600 9800
+Wire Notes Line
+	1250 9650 3600 9650
+Wire Notes Line
+	1250 10000 3600 10000
+Wire Notes Line
+	1600 9500 1600 10150
+Wire Notes Line
+	2100 9500 2100 10150
+Wire Notes Line
+	2800 9500 2800 10150
+Text Notes 1550 9350 0    60   ~ 0
+Подключение платы к интерфейсу SPI
 $EndSCHEMATC

Commit message: Поправил название микросхемы 74HC595B на 74HC595D.
Parts:
- DD1, DD2, DD3, DD4, DD5: value 74HC595B -> 74HC595D
Other:
- note added: "SPI SafeDuino SafeDuino 2560\n\nDS MOSI 11 MOSI\n\nSHCP SCK 13 SCK\n\nSTCP CS 8 8"
- note removed: "SPI SafeDuino SafeDuino 2560\n\nDS MOSI 14 MOSI\n\nSHCP SCK 13 SCK\n\nSTCP CS 8 8"
Changed lines of the file:
@@
 EESchema Schematic File Version 2
 LIBS:mod_16_segment_LED-cache
-EELAYER 27 0
+EELAYER 25 0
 EELAYER END
 $Descr A3 16535 11693
@@
 Sheet 1 1
 Title ""
-Date "21 jan 2016"
+Date "15 feb 2016"
 Rev ""
 Comp ""
@@
 P 5600 8200
 F 0 "DD5" H 5450 8750 70  0000 C CNN
-F 1 "74HC595B" H 5600 8600 70  0000 C CNN
+F 1 "74HC595D" H 5600 8600 70  0000 C CNN
 F 2 "" H 5600 8200 60  0001 C CNN
 F 3 "" H 5600 8200 60  0001 C CNN
@@
 P 5600 6500
 F 0 "DD4" H 5450 7050 70  0000 C CNN
-F 1 "74HC595B" H 5600 6900 70  0000 C CNN
+F 1 "74HC595D" H 5600 6900 70  0000 C CNN
 F 2 "" H 5600 6500 60  0001 C CNN
 F 3 "" H 5600 6500 60  0001 C CNN
@@
 P 5650 4850
 F 0 "DD3" H 5500 5400 70  0000 C CNN
-F 1 "74HC595B" H 5650 5250 70  0000 C CNN
+F 1 "74HC595D" H 5650 5250 70  0000 C CNN
 F 2 "" H 5650 4850 60  0001 C CNN
 F 3 "" H 5650 4850 60  0001 C CNN
@@
 P 5650 3200
 F 0 "DD2" H 5500 3750 70  0000 C CNN
-F 1 "74HC595B" H 5650 3600 70  0000 C CNN
+F 1 "74HC595D" H 5650 3600 70  0000 C CNN
 F 2 "" H 5650 3200 60  0001 C CNN
 F 3 "" H 5650 3200 60  0001 C CNN
@@
 P 5650 1600
 F 0 "DD1" H 5500 2150 70  0000 C CNN
-F 1 "74HC595B" H 5650 2000 70  0000 C CNN
+F 1 "74HC595D" H 5650 2000 70  0000 C CNN
 F 2 "" H 5650 1600 60  0001 C CNN
 F 3 "" H 5650 1600 60  0001 C CNN
@@
 	1    0    0    -1
 $EndComp
-Text Notes 1250 9600 0    60   ~ 0
-           SPI        SafeDuino    SafeDuino 2560\n\nDS        MOSI         14            MOSI\n\nSHCP      SCK         13             SCK\n\nSTCP       CS           8               8
+Text Notes 1200 10200 0    60   ~ 0
+           SPI        SafeDuino    SafeDuino 2560\n\nDS        MOSI         11            MOSI\n\nSHCP      SCK         13             SCK\n\nSTCP       CS           8               8
 Wire Notes Line
-	1250 9800 3600 9800
+	1200 9875 3550 9875
 Wire Notes Line
-	1250 9650 3600 9650
+	1200 9725 3550 9725
 Wire Notes Line
-	1250 10000 3600 10000
+	1200 10075 3550 10075
 Wire Notes Line
-	1600 9500 1600 10150
+	1550 9575 1550 10225
 Wire Notes Line
-	2100 9500 2100 10150
+	2050 9575 2050 10225
 Wire Notes Line
-	2800 9500 2800 10150
-Text Notes 1550 9350 0    60   ~ 0
+	2750 9575 2750 10225
+Text Notes 1325 9450 0    60   ~ 0
 Подключение платы к интерфейсу SPI
 $EndSCHEMATC
