File: modul_current_meter/modul_current_meter.sch (KiCad schematic (older format))
At the start: 9 parts

Commit message: Добавил проект платы измерителя тока.
Parts:
- R1, R2: footprint (none) -> IWsmd_case:SMD0805
Changed lines of the file:
@@
 	3800 2900 3800 3000
 Wire Wire Line
-	3700 3000 3800 3000
-Wire Wire Line
-	3800 3000 4350 3000
-Wire Wire Line
-	4350 3000 4450 3000
+	3700 3000 4450 3000
 Wire Wire Line
 	4350 3000 4350 2900
@@
 	3800 3250 3800 3350
 Wire Wire Line
-	3700 3350 3800 3350
-Wire Wire Line
-	3800 3350 4350 3350
-Wire Wire Line
-	4350 3350 4450 3350
+	3700 3350 4450 3350
 Wire Wire Line
 	4450 3250 4350 3250
@@
 	6750 3100 6750 3400
 Wire Wire Line
-	6200 3400 6750 3400
-Wire Wire Line
-	6750 3400 7050 3400
+	6200 3400 7050 3400
 Connection ~ 6750 3400
 Wire Wire Line
-	6200 3300 7200 3300
-Wire Wire Line
-	7200 3300 7650 3300
-Wire Wire Line
-	7650 3300 7900 3300
+	6200 3300 7900 3300
 Wire Wire Line
 	7200 3550 7200 3300
@@
 F 0 "R1" H 6350 3000 71  0000 C CNN
 F 1 "2 к" H 6750 3000 71  0000 C CNN
-F 2 "" H 6400 2900 60  0000 C CNN
+F 2 "IWsmd_case:SMD0805" H 6400 2900 60  0001 C CNN
 F 3 "" H 6400 2900 60  0000 C CNN
 	1    6400 2900
@@
 F 0 "R2" V 7400 2600 71  0000 C CNN
 F 1 "10 к" V 7300 2600 71  0000 C CNN
-F 2 "" H 7200 2800 60  0000 C CNN
+F 2 "IWsmd_case:SMD0805" H 7200 2800 60  0001 C CNN
 F 3 "" H 7200 2800 60  0000 C CNN
 	1    7200 2800
@@
 	6200 2900 6400 2900
 Wire Wire Line
-	6650 2900 7200 2900
-Wire Wire Line
-	7200 2900 7750 2900
+	6650 2900 7750 2900
 Wire Wire Line
 	7200 2800 7200 2900
