File: modul_encoder_ec11e/modul_encoder_ec11e.kicad_pcb (KiCad board)
At the start: 2 copper layers, 30 x 30 mm, 9 parts

Commit message: Перевёл плату энкодера под kicad 6.0. Добавли описание к с схемой и программой.
Other:
- net class Default removed
